File: bldcdriver/3halfbridge.kicad_sch (KiCad schematic)
At the start: 0 parts

Commit message: Created hierarchical sheets for every major component with a very basic block diagram on the front page
Parts:
- added Q1, Q2, Q3, Q4, Q5, Q6: IRF3205, Package_TO_SOT_THT:TO-220-3_Horizontal_TabDown, symbol Transistor_FET:IRF3205
- added R1, R2, R3: R, Resistor_SMD:R_0201_0603Metric, symbol Device:R
Connections:
- new net +24V: Q1.2 (D), Q3.2 (D), Q5.2 (D)
- new net GHA: Q1.1 (G)
- new net GHB: Q3.1 (G)
- new net GHC: Q5.1 (G)
- new net GLA: Q2.1 (G)
- new net GLB: Q4.1 (G)
- new net GLC: Q6.1 (G)
- new net GND: R1.2, R2.2, R3.2
- new net Phase A: Q1.3 (S), Q2.2 (D)
- new net Phase B: Q3.3 (S), Q4.2 (D)
- new net Phase C: Q5.3 (S), Q6.2 (D)
- new net SPA: Q2.3 (S), R1.1
- new net SPB: Q4.3 (S), R2.1
- new net SPC: Q6.3 (S), R3.1
Other:
- note added: "MOSFET Half Bridge"
