File: bldcdriver/power_bldc.kicad_sch (KiCad schematic)
At the start: 0 parts

Commit message: Added a USB C Connector and wired it up to act as USB 2.0
Parts:
- added D1: BAT54W, Package_TO_SOT_SMD:SOT-323_SC-70, symbol Diode:BAT54W
- added J1: USB_C_Receptacle_USB2.0_14P, symbol Connector:USB_C_Receptacle_USB2.0_14P
- added R4, R5: 5.1k, symbol Device:R
Connections:
- new net: J1.B5 (CC2), R4.1
- new net: J1.A5 (CC1), R5.1
- new net +5V: D1.3 (K)
- new net D+: J1.A6 (D+), J1.B6 (D+)
- new net D-: J1.A7 (D-), J1.B7 (D-)
- new net GND: J1.A1 (GND), J1.A12 (GND), J1.B1 (GND), J1.B12 (GND), J1.S1 (SHIELD), R4.2, R5.2
- new net VBUS: D1.1 (A), J1.A4 (VBUS), J1.A9 (VBUS), J1.B4 (VBUS), J1.B9 (VBUS)
