File: bldcdriver/drv_bldc.kicad_sch (KiCad schematic)
At the start: 7 parts, among them U1 DRV8304SRHAR

Commit message: Finished DRV side fully, RP2040 almost fully done, FOC sensorless and sensor parts and power parts are left
Parts:
- added J2: Conn_01x03_Pin, symbol Connector:Conn_01x03_Pin
- added R8: R, symbol Device:R_Small
Connections:
- net +3.3V: now also R8.2
- net at U1.21 (SOC): now also J2.1 (Pin_1)
- net at U1.22 (SOB): now also J2.2 (Pin_2)
- net at U1.23 (SOA): now also J2.3 (Pin_3)
- net nFAULT: now reaches U1.25 (FAULT_N)
- net nFAULT: now also R8.1
- net SPI_SDI: now reaches U1.26 (SDO)
- net SPI_SDO: now reaches U1.27 (SDI)
- net SPI_CLK: now reaches U1.28 (SCLK)
- net SPI_CSn: now reaches U1.29 (SCS_N)
- net DREN: now reaches U1.30 (ENABLE)
- net INHA: now reaches U1.34 (INHA)
- net INLA: now reaches U1.35 (INLA)
- net INHB: now reaches U1.36 (INHB)
- net INLB: now reaches U1.37 (INLB)
- net INHC: now reaches U1.38 (INHC)
- net INLC: now reaches U1.39 (INLC)
